File: ORBITAL Board/ORBITAL Board.kicad_sch (KiCad schematic)
At the start: 64 parts

Commit message: Uploading Board Progress
Parts:
- removed AE? (x2): Antenna, symbol Device:Antenna
- removed U?: PX1172RH, symbol Compon:PX1172RH
- added AE1, AE2: Antenna, GPS:SMA_Molex_73251-1153_EdgeMount_Horizontal, symbol Device:Antenna
- added C1: 22n, Capacitor_SMD:C_0402_1005Metric, symbol Device:C
- added C19: 22p, Capacitor_SMD:C_0402_1005Metric_Pad0.74x0.62mm_HandSolder, symbol Device:C_Small
- added C2: 10u, Capacitor_SMD:C_0402_1005Metric, symbol Device:C
- added C21: 22u, Capacitor_SMD:C_0402_1005Metric_Pad0.74x0.62mm_HandSolder, symbol Device:C_Small
- added C24, C3, C39: 100n, Capacitor_SMD:C_0402_1005Metric_Pad0.74x0.62mm_HandSolder, symbol Device:C_Small
- added C25: 10n, Capacitor_SMD:C_0402_1005Metric, symbol Device:C
- added C27: 1n, Capacitor_SMD:C_0402_1005Metric, symbol Device:C
- added C33: 2.2u, Capacitor_SMD:C_0402_1005Metric, symbol Device:C_Small
- added C35: 22u, Capacitor_SMD:C_0402_1005Metric, symbol Device:C_Small
- added L1: 4.7u, Inductor_SMD:L_0603_1608Metric, symbol Device:L
- added L3, L4: 39n, Inductor_SMD:L_0603_1608Metric, symbol Device:L
- added R11: 225k, Resistor_SMD:R_0603_1608Metric, symbol Device:R
- added R16: 100K, Resistor_SMD:R_0603_1608Metric, symbol Device:R
- added R17: 50k, Resistor_SMD:R_0603_1608Metric, symbol Device:R
- added R18, R19: 18, Resistor_SMD:R_0603_1608Metric, symbol Device:R
- added R20: 1K, Resistor_SMD:R_0603_1608Metric, symbol Device:R_Small
- added R21: 47K, Resistor_SMD:R_0603_1608Metric, symbol Device:R_Small
- added R24, R25: .33, Resistor_SMD:R_0603_1608Metric, symbol Device:R_Small
- added R3: 350K, Resistor_SMD:R_0603_1608Metric, symbol Device:R_Small
- added R4: 510K, Resistor_SMD:R_0603_1608Metric, symbol Device:R_Small
- added RB1, RB2: 100K, Resistor_SMD:R_0603_1608Metric, symbol Device:R_Small
- added U1: PTPS563206DRLR, footprints:SOT_07SDRLR_TEX, symbol 2024-02-23_21-01-39:PTPS563206DRLR
- added U7: ~, GPS:PX1172RH, symbol GPS:PX1172RH
- C10, C11, C12, C13, C15, C16, C7, C9: renamed from C?; footprint (none) -> Capacitor_SMD:C_0402_1005Metric
- C14: renamed from C?; value 47u -> 100u; footprint (none) -> Capacitor_SMD:C_0402_1005Metric
- C6: renamed from C?; footprint (none) -> Capacitor_SMD:C_0402_1005Metric_Pad0.74x0.62mm_HandSolder
- C8: renamed from C?; value 0 -> 1.8n; footprint (none) -> Capacitor_SMD:C_0402_1005Metric
- D1: renamed from D?; footprint (none) -> Diode_SMD:D_0603_1608Metric
- L2: renamed from L?; value L_Small -> 3.3u; footprint (none) -> Inductor_SMD:L_0603_1608Metric
- R1: renamed from R?; value R_Small -> 500K; footprint (none) -> Resistor_SMD:R_0603_1608Metric
- R10: renamed from R?; value R_Small -> 40.2K; footprint (none) -> Resistor_SMD:R_0603_1608Metric
- R12, R13, R14: renamed from R?; value R_Small -> 5.1K; footprint (none) -> Resistor_SMD:R_0603_1608Metric
- R2: renamed from R?; value R_Small -> 100K; footprint (none) -> Resistor_SMD:R_0603_1608Metric
- gave numbers to parts that had none: 42
Connections:
- net ENV_SCL is gone; now on net D1: R28.1, U8.8 (SCLK)
- net ENV_SDA is gone; now on net D0: R27.2, U8.7 (SDI/SDA)
- net +3.3V: now also C19.1, C21.2, C24.2, L1.2, L3.2, L4.2, R11.2, R18.2, R19.2, U7.33 (VDD33), U7.34 (VDD33)
- net A3: now also U6.11 (REF)
- net D4: now also U6.1 (DIR)
- net D5: now also U6.2 (STCK)
- net D6: now also U6.13 (EN/FLT), C25.1, R18.1
- net D7: now also U6.14 (STBY/RESET), C27.1, R19.1
- net D8: now also U7.16 (RXD_R)
- net D9: now also U7.17 (TXD_R)
- net GND: now also U6.17 (EPAD), U6.7 (GND), C1.2, C2.1, C21.1, C24.1, C25.2, C27.2, C33.2, C35.2, C39.2, R17.1, R21.2, R24.2, R25.2, RB1.1, RB2.1, U1.3 (GND), U7.1 (GND), U7.1$ (GND), U7.12 (GND), U7.14 (GND), U7.3 (GND), U7.32 (GND), U7.48 (GND); no longer C10.1
- net VBUS: now also C10.1, R3.2, R4.2
- net V_BCK: now also U7.36 (V_BCKP)
- net at U6.12 (TOFF): now also R20.1, R21.1
- net at U6.4 (SENSEA): now also R24.1
- net +6V: now reaches U6.6 (VS)
- net +6V: now also C14.1, R1.2, R12.2, R13.2, R14.2, U4. (VOUT), C2.2, C33.1, C35.1, C39.1, R16.2, U1.1 (VIN)
- net at U6.9 (SENSEB): now also R25.1
- removed net +5V: C14.1, R1.2, R12.2, R13.2, R14.2, U4. (VOUT)
- new net: C3.2, L1.1, U1.2 (SW)
- new net: AE2.1 (A), L3.1, U7.13 (RF_IN2)
- new net: AE1.1 (A), L4.1, U7.2 (RF_INI)
- new net: C19.2, R11.1, R17.2, U1.6 (FB)
- new net: C3.1, U1.4 (BST)
- new net: R3.1, RB1.2, U4. (VOUT)
- new net: R4.1, RB2.2, U4. (VOUT)
- new net: R16.1, U1.5 (EN)
- new net: C1.1, R20.2
Other:
- note added: "Motor Connect Pins"
- note added: "Note: Vout = .6*(1+(R11/R17) = .6 + (1+(225K/50K)) = 3.3V"
- note added: "Note: Vout = 1 + (R1/R2) = 1 + (500K/100K) = 6V"
- note added: "Stepper Motor"
- moved on the sheet: C17, C18, C20, C22, C23, C28, C29, C30, C31, C32, C34, C36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

Commit message: Adding schematic and PCB updates
Parts:
- removed C16: 22U, Capacitor_SMD:C_0402_1005Metric, symbol Device:C_Small
- added C41: 22u, Capacitor_SMD:C_0603_1608Metric, symbol Device:C_Small
- BT1: footprint (none) -> BackupBattery:BAT_MS920SE-FL27E
- C13, C15: value .1u -> 100n
- C6: value 22U -> 22u; footprint Capacitor_SMD:C_0402_1005Metric_Pad0.74x0.62mm_HandSolder -> Capacitor_SMD:C_0603_1608Metric
- D1: value D_Small -> D_Zener; footprint Diode_SMD:D_0603_1608Metric -> GPS:DIO_RB400DFH_ROM-M
- Y1: footprint (none) -> Crystal:Crystal_SMD_Abracon_ABM8G-4Pin_3.2x2.5mm
Connections:
- net +BATT: now also C41.1
- net GND: now also C6.1, C41.2; no longer C6.2
- net VBUS: now also C6.2; no longer C6.1
Other:
- moved on the sheet: C14
Changed lines of the file:
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@@
   (junction (at 132.08 52.07) (diameter 0) (color 0 0 0 0)
   )
+  (junction (at 168.91 39.37) (diameter 0) (color 0 0 0 0)
+  )
   (junction (at 294.64 24.13) (diameter 0) (color 0 0 0 0)
   )
@@
   (junction (at 361.95 27.94) (diameter 0) (color 0 0 0 0)
   )
-  (junction (at 168.91 39.37) (diameter 0) (color 0 0 0 0)
-  )
   (junction (at 264.16 151.13) (diameter 0) (color 0 0 0 0)
   )
@@
     (stroke (width 0) (type default))
   )
+  (wire (pts (xy 168.91 24.13) (xy 168.91 33.02))
+    (stroke (width 0) (type default))
+  )
   (wire (pts (xy 134.62 49.53) (xy 134.62 52.07))
     (stroke (width 0) (type default))
@@
     (stroke (width 0) (type default))
   )
-  (wire (pts (xy 168.91 34.29) (xy 168.91 24.13))
-    (stroke (width 0) (type default))
-  )
   (wire (pts (xy 121.92 113.03) (xy 121.92 118.11))
     (stroke (width 0) (type default))
@@
     (stroke (width 0) (type default))
   )
+  (wire (pts (xy 168.91 38.1) (xy 168.91 39.37))
+    (stroke (width 0) (type default))
+  )
   (wire (pts (xy 217.17 142.24) (xy 217.17 146.05))
     (stroke (width 0) (type default))
@@
     (stroke (width 0) (type default))
   )
+  (wire (pts (xy 166.37 58.42) (xy 166.37 57.15))
+    (stroke (width 0) (type default))
+  )
   (wire (pts (xy 21.59 59.69) (xy 29.21 59.69))
     (stroke (width 0) (type default))
@@
     (stroke (width 0) (type default))
   )
+  (wire (pts (xy 166.37 53.34) (xy 166.37 52.07))
+    (stroke (width 0) (type default))
+  )
   (wire (pts (xy 378.46 142.24) (xy 375.92 142.24))
     (stroke (width 0) (type default))
@@
     (stroke (width 0) (type default))
   )
+  (wire (pts (xy 168.91 39.37) (xy 172.72 39.37))
+    (stroke (width 0) (type default))
+  )
   (wire (pts (xy 381 71.12) (xy 384.81 71.12))
     (stroke (width 0) (type default))
@@
     (stroke (width 0) (type default))
   )
-  (wire (pts (xy 106.68 44.45) (xy 106.68 52.07))
+  (wire (pts (xy 106.68 48.26) (xy 106.68 52.07))
     (stroke (width 0) (type default))
   )
@@
     (stroke (width 0) (type default))
   )
+  (wire (pts (xy 106.68 43.18) (xy 106.68 39.37))
+    (stroke (width 0) (type default))
+  )
   (wire (pts (xy 162.56 45.72) (xy 165.1 45.72))
     (stroke (width 0) (type default))
@@
       (effects (font (size 1.27 1.27)) (justify left))
     )
-    (property "Value" ".1u" (at 167.64 43.18 0)
+    (property "Value" "100n" (at 167.64 43.18 0)
       (effects (font (size 1.27 1.27)) (justify left))
     )
@@
       (effects (font (size 1.27 1.27)) (justify left))
     )
-    (property "Value" ".1u" (at 170.18 48.26 0)
+    (property "Value" "100n" (at 170.18 48.26 0)
       (effects (font (size 1.27 1.27)) (justify left))
     )
@@
       (effects (font (size 1.27 1.27)) (justify left))
     )
-    (property "Footprint" "" (at 190.5 218.44 0)
+    (property "Footprint" "Crystal:Crystal_SMD_Abracon_ABM8G-4Pin_3.2x2.5mm" (at 190.5 218.44 0)
       (effects (font (size 1.27 1.27)) hide)
     )
@@
     )
   )
+  (symbol (lib_name "C_Small_1") (lib_id "Device:C_Small") (at 168.91 35.56 180) (unit 1)
+    (in_bom yes) (on_board yes) (dnp no)
+    (property "Reference" "C41" (at 168.91 33.02 0)
+      (effects (font (size 1.27 1.27)) (justify right))
+    )
+    (property "Value" "22u" (at 171.45 36.83 0)
+      (effects (font (size 1.27 1.27)) (justify right))
+    )
+    (property "Footprint" "Capacitor_SMD:C_0603_1608Metric" (at 168.91 35.56 0)
+      (effects (font (size 1.27 1.27)) hide)
+    )
+    (property "Datasheet" "~" (at 168.91 35.56 0)
+      (effects (font (size 1.27 1.27)) hide)
+    )
+    (pin "1")
+    (pin "2")
+    (instances
+      (project "ORBITAL Board"
+        (path "/ed00f797-6c76-4d28-b3bc-c732d14de183"
+          (reference "C41") (unit 1)
+        )
+      )
+    )
+  )
   (symbol (lib_id "power:+3V3") (at 335.28 233.68 90) (unit 1)
     (in_bom yes) (on_board yes) (dnp no) (fields_autoplaced)
@@
     )
   )
-  (symbol (lib_name "C_Small_1") (lib_id "Device:C_Small") (at 106.68 41.91 0) (unit 1)
-    (in_bom yes) (on_board yes) (dnp no) (fields_autoplaced)
-    (property "Reference" "C6" (at 109.22 40.6463 0)
-      (effects (font (size 1.27 1.27)) (justify left))
-    )
-    (property "Value" "22U" (at 109.22 43.1863 0)
-      (effects (font (size 1.27 1.27)) (justify left))
-    )
-    (property "Footprint" "Capacitor_SMD:C_0402_1005Metric_Pad0.74x0.62mm_HandSolder" (at 106.68 41.91 0)
-      (effects (font (size 1.27 1.27)) hide)
-    )
-    (property "Datasheet" "~" (at 106.68 41.91 0)
-      (effects (font (size 1.27 1.27)) hide)
-    )
-    (pin "1")
-    (pin "2")
-    (instances
-      (project "ORBITAL Board"
-        (path "/ed00f797-6c76-4d28-b3bc-c732d14de183"
-          (reference "C6") (unit 1)
-        )
-      )
-    )
-  )
   (symbol (lib_name "C_Small_1") (lib_id "Device:C_Small") (at 129.54 107.95 0) (unit 1)
     (in_bom yes) (on_board yes) (dnp no) (fields_autoplaced)
@@
     )
   )
-  (symbol (lib_id "Device:C_Small") (at 166.37 54.61 0) (unit 1)
+  (symbol (lib_name "C_Small_1") (lib_id "Device:C_Small") (at 106.68 45.72 180) (unit 1)
+    (in_bom yes) (on_board yes) (dnp no)
+    (property "Reference" "C6" (at 106.68 43.18 0)
+      (effects (font (size 1.27 1.27)) (justify right))
+    )
+    (property "Value" "22u" (at 106.68 49.53 0)
+      (effects (font (size 1.27 1.27)) (justify right))
+    )
+    (property "Footprint" "Capacitor_SMD:C_0603_1608Metric" (at 106.68 45.72 0)
+      (effects (font (size 1.27 1.27)) hide)
+    )
+    (property "Datasheet" "~" (at 106.68 45.72 0)
+      (effects (font (size 1.27 1.27)) hide)
+    )
+    (pin "1")
+    (pin "2")
+    (instances
+      (project "ORBITAL Board"
+        (path "/ed00f797-6c76-4d28-b3bc-c732d14de183"
+          (reference "C6") (unit 1)
+        )
+      )
+    )
+  )
+  (symbol (lib_id "Device:C_Small") (at 166.37 55.88 0) (unit 1)
     (in_bom yes) (on_board yes) (dnp no) (fields_autoplaced)
-    (property "Reference" "C14" (at 168.91 53.3463 0)
+    (property "Reference" "C14" (at 168.91 54.6163 0)
       (effects (font (size 1.27 1.27)) (justify left))
     )
-    (property "Value" "100u" (at 168.91 55.8863 0)
+    (property "Value" "100u" (at 168.91 57.1563 0)
       (effects (font (size 1.27 1.27)) (justify left))
     )
-    (property "Footprint" "Capacitor_SMD:C_0402_1005Metric" (at 166.37 54.61 0)
+    (property "Footprint" "Capacitor_SMD:C_0402_1005Metric" (at 166.37 55.88 0)
       (effects (font (size 1.27 1.27)) hide)
     )
-    (property "Datasheet" "~" (at 166.37 54.61 0)
+    (property "Datasheet" "~" (at 166.37 55.88 0)
       (effects (font (size 1.27 1.27)) hide)
     )
@@
       (effects (font (size 1.27 1.27)) (justify left))
     )
-    (property "Footprint" "" (at 22.86 107.696 90)
+    (property "Footprint" "BackupBattery:BAT_MS920SE-FL27E" (at 22.86 107.696 90)
       (effects (font (size 1.27 1.27)) hide)
     )
@@
     )
   )
-  (symbol (lib_id "power:+BATT") (at 168.91 39.37 270) (unit 1)
+  (symbol (lib_id "power:+BATT") (at 172.72 39.37 270) (unit 1)
     (in_bom yes) (on_board yes) (dnp no)
-    (property "Reference" "#PWR0112" (at 165.1 39.37 0)
+    (property "Reference" "#PWR0112" (at 168.91 39.37 0)
       (effects (font (size 1.27 1.27)) hide)
     )
-    (property "Value" "+BATT" (at 176.53 39.37 90)
+    (property "Value" "+BATT" (at 179.07 39.37 90)
       (effects (font (size 1.27 1.27)))
     )
-    (property "Footprint" "" (at 168.91 39.37 0)
+    (property "Footprint" "" (at 172.72 39.37 0)
       (effects (font (size 1.27 1.27)) hide)
     )
-    (property "Datasheet" "" (at 168.91 39.37 0)
+    (property "Datasheet" "" (at 172.72 39.37 0)
       (effects (font (size 1.27 1.27)) hide)
     )
@@
   (symbol (lib_id "Device:D_Small") (at 22.86 93.98 90) (unit 1)
     (in_bom yes) (on_board yes) (dnp no) (fields_autoplaced)
-    (property "Reference" "D1" (at 25.4 92.7099 90)
+    (property "Reference" "D1" (at 25.4 92.71 90)
       (effects (font (size 1.27 1.27)) (justify right))
     )
-    (property "Value" "D_Small" (at 25.4 95.2499 90)
+    (property "Value" "D_Zener" (at 25.4 95.25 90)
       (effects (font (size 1.27 1.27)) (justify right))
     )
-    (property "Footprint" "Diode_SMD:D_0603_1608Metric" (at 22.86 93.98 90)
+    (property "Footprint" "GPS:DIO_RB400DFH_ROM-M" (at 22.86 93.98 90)
       (effects (font (size 1.27 1.27)) hide)
     )
@@
         )
       )
-    )
-  )
-  (symbol (lib_id "Device:C_Small") (at 168.91 36.83 0) (unit 1)
-    (in_bom yes) (on_board yes) (dnp no)
-    (property "Reference" "C16" (at 171.45 35.5662 0)
-      (effects (font (size 1.27 1.27)) (justify left))
-    )
-    (property "Value" "22U" (at 163.83 36.83 0)
-      (effects (font (size 1.27 1.27)) (justify left))
-    )
-    (property "Footprint" "Capacitor_SMD:C_0402_1005Metric" (at 168.91 36.83 0)
-      (effects (font (size 1.27 1.27)) hide)
-    )
-    (property "Datasheet" "~" (at 168.91 36.83 0)
-      (effects (font (size 1.27 1.27)) hide)
-    )
-    (pin "1")
-    (pin "2")
-    (instances
-      (project "ORBITAL Board"
-        (path "/ed00f797-6c76-4d28-b3bc-c732d14de183"
-          (reference "C16") (unit 1)
-        )
-      )

Commit message: Updating board + adding in board notes
Connections:
- net GND: now also U7.37 (GND), U7.41 (GND)
Changed lines of the file:
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@@
       (effects (font (size 1.27 1.27)) hide)
     )
-    (property "Datasheet" "" (at 431.8 50.8 0)
+    (property "Datasheet" "https://navspark.mybigcommerce.com/content/PX1172RH_DS.pdf" (at 431.8 50.8 0)
       (effects (font (size 1.27 1.27)) hide)
     )
@@
     )
   )
+  (symbol (lib_id "power:GND") (at 351.79 27.94 180) (unit 1)
+    (in_bom yes) (on_board yes) (dnp no) (fields_autoplaced)
+    (property "Reference" "#PWR023" (at 351.79 21.59 0)
+      (effects (font (size 1.27 1.27)) hide)
+    )
+    (property "Value" "GND" (at 351.79 22.86 0)
+      (effects (font (size 1.27 1.27)))
+    )
+    (property "Footprint" "" (at 351.79 27.94 0)
+      (effects (font (size 1.27 1.27)) hide)
+    )
+    (property "Datasheet" "" (at 351.79 27.94 0)
+      (effects (font (size 1.27 1.27)) hide)
+    )
+    (pin "1")
+    (instances
+      (project "ORBITAL Board"
+        (path "/ed00f797-6c76-4d28-b3bc-c732d14de183"
+          (reference "#PWR023") (unit 1)
+        )
+      )
+    )
+  )
   (symbol (lib_id "power:GND") (at 166.37 57.15 0) (unit 1)
     (in_bom yes) (on_board yes) (dnp no)
@@
         )
       )
+    )
+  )
+  (symbol (lib_id "power:GND") (at 346.71 27.94 180) (unit 1)
+    (in_bom yes) (on_board yes) (dnp no) (fields_autoplaced)
+    (property "Reference" "#PWR024" (at 346.71 21.59 0)
+      (effects (font (size 1.27 1.27)) hide)
+    )
+    (property "Value" "GND" (at 346.71 22.86 0)
+      (effects (font (size 1.27 1.27)))
+    )
+    (property "Footprint" "" (at 346.71 27.94 0)
+      (effects (font (size 1.27 1.27)) hide)
+    )
+    (property "Datasheet" "" (at 346.71 27.94 0)
+      (effects (font (size 1.27 1.27)) hide)
+    )
+    (pin "1")
+    (instances
+      (project "ORBITAL Board"
+        (path "/ed00f797-6c76-4d28-b3bc-c732d14de183"
+          (reference "#PWR024") (unit 1)
+        )
+      )
